Commit message: Added 2 more legs and moved all legs to two sides. Need to add two more legs but this is looking very promising"

File: urdf/body.urdf (robot description, URDF)
Before this commit: robot robot, 13 links, 12 joints
Joints:
- joint Torso_BackLeg: origin xyz=0 -0.5 2 rpy=0 0 0 -> xyz=0.2 -0.5 2 rpy=0 0 0
- joint Torso_FrontLeg: origin xyz=0 0.5 2 rpy=0 0 0 -> xyz=0.2 0.5 2 rpy=0 0 0

Commit message: Removed runway and obsticles

File: urdf/body.urdf (robot description, URDF)
Before this commit: robot robot, 13 links, 12 joints
Links:
- added link BackMiddleRightLeg, mass 1; collision box size=0.2 1 0.2; visual box size=0.2 1 0.2
- added link BackMiddleRightLowerLeg, mass 1; collision box size=0.2 0.2 1; visual box size=0.2 0.2 1
- added link FrontMiddleRightLeg, mass 1; collision box size=0.2 1 0.2; visual box size=0.2 1 0.2
- added link FrontMiddleRightLowerLeg, mass 1; collision box size=0.2 0.2 1; visual box size=0.2 0.2 1
Joints:
- added joint BackMiddleRightLeg_BackMiddleRightLowerLeg: type revolute, parent BackMiddleRightLeg, child BackMiddleRightLowerLeg, origin xyz=0 -1 0 rpy=0 0 0, axis 1 0 0, limit lower=-3.14159 upper=3.14159 effort=0.0 velocity=0.0
- added joint FrontMiddleRightLeg_FrontMiddleRightLowerLeg: type revolute, parent FrontMiddleRightLeg, child FrontMiddleRightLowerLeg, origin xyz=0 1 0 rpy=0 0 0, axis 1 0 0, limit lower=-3.14159 upper=3.14159 effort=0.0 velocity=0.0
- added joint Torso_BackMiddleRightLeg: type revolute, parent Torso, child BackMiddleRightLeg, origin xyz=-0.2 -0.5 1 rpy=0 0 0, axis 0 0 1, limit lower=-3.14159 upper=3.14159 effort=0.0 velocity=0.0
- added joint Torso_FrontMiddleRightLeg: type revolute, parent Torso, child FrontMiddleRightLeg, origin xyz=-0.2 0.5 1 rpy=0 0 0, axis 0 0 1, limit lower=-3.14159 upper=3.14159 effort=0.0 velocity=0.0
- joint Torso_BackLeftLeg: origin xyz=0.5 0.5 2 rpy=0 0 0 -> xyz=0.5 0.5 1 rpy=0 0 0
- joint Torso_BackLeg: origin xyz=0.2 -0.5 2 rpy=0 0 0 -> xyz=0.2 -0.5 1 rpy=0 0 0
- joint Torso_BackRightLeg: origin xyz=0.5 -0.5 2 rpy=0 0 0 -> xyz=0.5 -0.5 1 rpy=0 0 0
- joint Torso_FrontLeftLeg: origin xyz=-0.5 0.5 2 rpy=0 0 0 -> xyz=-0.5 0.5 1 rpy=0 0 0
- joint Torso_FrontLeg: origin xyz=0.2 0.5 2 rpy=0 0 0 -> xyz=0.2 0.5 1 rpy=0 0 0
- joint Torso_FrontRightLeg: origin xyz=-0.5 -0.5 2 rpy=0 0 0 -> xyz=-0.5 -0.5 1 rpy=0 0 0
